Commit message: visual_features_extractor: new way for calculation of distance to features. Added distance input  in the service set_desired_template visual_servoing_... renamed to imbvs_with_obstacles_avoidance. In addition made a smoothing of a distance to obstacles. Addded new lwr configuration for HRI as hri_lwr Improved support for an extrinsic calibration based on aruco in kinect_fusion 	modified:   eye-in-hand/visual_features_extractor/CMakeLists.txt 	modified:   eye-in-hand/visual_features_extractor/include/visual_features_extractor/visual_features_extractor.h 	modified:   eye-in-hand/visual_features_extractor/launch/visual_features_extractor.launch 	modified:   eye-in-hand/visual_features_extractor/src/visual_features_extractor.cpp 	new file:   eye-in-hand/visual_features_extractor/srv/set_depth.srv 	modified:   eye-to-hand/kinect_fusion/include/kinect_fusion/kinect_fusion.h 	new file:   eye-to-hand/kinect_fusion/launch/hri_kinect_fusion.launch 	new file:   eye-to-hand/kinect_fusion/launch/ics_kinect_fusion.launch 	modified:   eye-to-hand/kinect_fusion/src/kinect_fusion.cpp 	new file:   eye-to-hand/obstacle_detector/config/hri_parameters.yaml 	new file:   eye-to-hand/obstacle_detector/config/ics_parameters.yaml 	modified:   eye-to-hand/obstacle_detector/launch/obstacle_detector.launch 	modified:   eye-to-hand/obstacle_detector/src/obstacle_detector.cpp 	renamed:    visual-servoing-with-safe-interaction/.gitignore -> imbvs_with_obstacles_avoidance/.gitignore 	renamed:    visual-servoing-with-safe-interaction/CMakeLists.txt -> imbvs_with_obstacles_avoidance/CMakeLists.txt 	new file:   imbvs_with_obstacles_avoidance/README.md 	renamed:    visual-servoing-with-safe-interaction/include/visual_servoing_with_safe_interaction/visual_servoing_with_safe_interaction.h -> imbvs_with_obstacles_avoidance/include/imbvs_with_obstacles_avoidance/imbvs_with_obstacles_avoidance.h 	renamed:    visual-servoing-with-safe-interaction/include/utils/pseudo_inversion.h -> imbvs_with_obstacles_avoidance/include/utils/pseudo_inversion.h 	renamed:    visual-servoing-with-safe-interaction/include/utils/skew_symmetric.h -> imbvs_with_obstacles_avoidance/include/utils/skew_symmetric.h 	renamed:    visual-servoing-with-safe-interaction/include/utils/trajectrory_splines.h -> imbvs_with_obstacles_avoidance/include/utils/trajectrory_splines.h 	renamed:    visual-servoing-with-safe-interaction/launch/visual_servoing_with_safe_interaction.launch -> imbvs_with_obstacles_avoidance/launch/imbvs_with_obstacles_avodance.launch 	renamed:    visual-servoing-with-safe-interaction/msg/ObsData.msg -> imbvs_with_obstacles_avoidance/msg/ObsData.msg 	renamed:    visual-servoing-with-safe-interaction/msg/PoseRPY.msg -> imbvs_with_obstacles_avoidance/msg/PoseRPY.msg 	renamed:    visual-servoing-with-safe-interaction/msg/RPY.msg -> imbvs_with_obstacles_avoidance/msg/RPY.msg 	renamed:    visual-servoing-with-safe-interaction/msg/VisFeature.msg -> imbvs_with_obstacles_avoidance/msg/VisFeature.msg 	renamed:    visual-servoing-with-safe-interaction/msg/VisualServoing.msg -> imbvs_with_obstacles_avoidance/msg/VisualServoing.msg 	renamed:    visual-servoing-with-safe-interaction/nodes/visual_servoing_with_safe_interaction_node.cpp -> imbvs_with_obstacles_avoidance/nodes/imbvs_with_obstacles_avoidance_node.cpp 	renamed:    visual-servoing-with-safe-interaction/package.xml -> imbvs_with_obstacles_avoidance/package.xml 	renamed:    visual-servoing-with-safe-interaction/src/visual_servoing_with_safe_interaction.cpp -> imbvs_with_obstacles_avoidance/src/imbvs_with_obstacles_avoidance.cpp 	renamed:    visual-servoing-with-safe-interaction/srv/SetTF.srv -> imbvs_with_obstacles_avoidance/srv/SetDepth.srv~ 	renamed:    visual-servoing-with-safe-interaction/srv/SetGama.srv -> imbvs_with_obstacles_avoidance/srv/SetGama.srv 	new file:   imbvs_with_obstacles_avoidance/srv/SetTF.srv 	new file:   kuka-lwr/hri_lwr/README.md 	new file:   kuka-lwr/hri_lwr/hri_lwr/CMakeLists.txt 	new file:   kuka-lwr/hri_lwr/hri_lwr/package.xml 	new file:   kuka-lwr/hri_lwr/hri_lwr_launch/CMakeLists.txt 	new file:   kuka-lwr/hri_lwr/hri_lwr_launch/launch/hri_lwr.launch 	new file:   kuka-lwr/hri_lwr/hri_lwr_launch/launch/rviz_config.rviz 	new file:   kuka-lwr/hri_lwr/hri_lwr_launch/package.xml 	new file:   kuka-lwr/hri_lwr/hri_lwr_setup/CMakeLists.txt 	new file:   kuka-lwr/hri_lwr/hri_lwr_setup/config/980067-FRI-Driver.init 	new file:   kuka-lwr/hri_lwr/hri_lwr_setup/config/controllers.yaml 	new file:   kuka-lwr/hri_lwr/hri_lwr_setup/config/hw_interface.yaml 	new file:   kuka-lwr/hri_lwr/hri_lwr_setup/config/load_start_position.yaml 	new file:   kuka-lwr/hri_lwr/hri_lwr_setup/config/t1_joint_limits.yaml 	new file:   kuka-lwr/hri_lwr/hri_lwr_setup/enviroment/hri_lwr_enviroment.urdf.xacro 	new file:   kuka-lwr/hri_lwr/hri_lwr_setup/package.xml 	new file:   kuka-lwr/hri_lwr/hri_lwr_setup/worlds/simple_environment.world 	new file:   kuka-lwr/ics_lwr/ics_lwr_launch/launch/hri_lwr.launch 	modified:   kuka-lwr/ics_lwr/ics_lwr_launch/launch/ics_lwr.launch 	modified:   kuka-lwr/ics_lwr/ics_lwr_launch/launch/rviz_config.rviz 	modified:   kuka-lwr/ics_lwr/ics_lwr_setup/config/hw_interface.yaml 	modified:   kuka-lwr/ics_lwr/ics_lwr_setup/enviroment/ics_lwr_enviroment.urdf.xacro 	modified:   kuka-lwr/lwr_description/model/kuka_lwr.urdf.xacro 	modified:   kuka-lwr/lwr_hw/src/lwr_hw/lwr_hw.cpp 	modified:   kuka-lwr/lwr_hw/src/lwr_hw/lwr_hw_gazebo.cpp 	deleted:    visual-servoing-with-safe-interaction/README.md

File: kuka-lwr/ics_lwr/ics_lwr_setup/enviroment/ics_lwr_enviroment.urdf.xacro (robot description, xacro)
@@ -156,9 +156,9 @@
     <xacro:property name="robot_origin_y" value="${panel_origin_y - panel_size_y/2}" />
     <xacro:property name="robot_origin_z" value="${panel_origin_z}" />
-    <xacro:property name="robotOriginR" value="${PI/2}" />
-    <xacro:property name="robotOriginP" value="${-PI/2}" />
+    <xacro:property name="robot_origin_roll" value="${PI/2}" />
+    <xacro:property name="robot_origin_pitch" value="${-PI/2}" />
     <xacro:property name="robot_origin_yaw" value="0" />
     <xacro:kuka_lwr parent="panel" name="lwr">
-        <origin xyz="${robot_origin_x} ${robot_origin_y} ${robot_origin_z}" rpy="${robotOriginR} ${robotOriginP} ${robot_origin_yaw}"/>
+        <origin xyz="${robot_origin_x} ${robot_origin_y} ${robot_origin_z}" rpy="${robot_origin_roll} ${robot_origin_pitch} ${robot_origin_yaw}"/>
     </xacro:kuka_lwr>
 </robot>

File: kuka-lwr/lwr_description/model/kuka_lwr.urdf.xacro (robot description, xacro)
@@ -9,9 +9,9 @@
 	<xacro:include filename="$(find lwr_description)/model/kuka_lwr.transmission.xacro"/>
 	<!-- properties /-->
-    <xacro:property name="base_mass" value="2.0"/>
+        <xacro:property name="base_mass" value="2.0"/>
         <xacro:property name="link_mass" value="2.35"/>
         <xacro:property name="wrist_mass" value="2.1"/>     <!-- 1.1 /-->
         <xacro:property name="tip_mass" value="2.25"/>      <!-- 0.25 /-->
-        <xacro:property name="velocity_scale" value="0.1"/>
+        <xacro:property name="velocity_scale" value="0.15"/>
         <xacro:property name="effort_scale" value="1"/>
 	<!-- URDF model /-->
