Commit message: Small fixes in lwr_hw, updated lwr_description, updated nodelet names in launch files 	modified:   eye-in-hand/visual_features_extractor/CMakeLists.txt 	modified:   eye-in-hand/visual_features_extractor/launch/visual_features_extractor.launch 	modified:   eye-in-hand/visual_features_extractor/src/visual_features_extractor.cpp 	modified:   eye-to-hand/kinect_fusion/CMakeLists.txt 	modified:   eye-to-hand/kinect_fusion/launch/hri_kinect_fusion.launch 	modified:   eye-to-hand/kinect_fusion/launch/ics_kinect_fusion.launch 	modified:   eye-to-hand/kinect_fusion/src/kinect_fusion.cpp 	modified:   eye-to-hand/obstacle_detector/CMakeLists.txt 	modified:   eye-to-hand/obstacle_detector/launch/obstacle_detector.launch 	deleted:    imbvs_with_obstacles_avoidance/launch/imbvs_with_obstacles_avodance.launch~ 	modified:   kuka-lwr/hri_lwr/hri_lwr_launch/launch/hri_lwr.launch 	deleted:    kuka-lwr/ics_lwr/ics_lwr_launch/launch/hri_lwr.launch 	modified:   kuka-lwr/ics_lwr/ics_lwr_launch/launch/ics_lwr.launch 	modified:   kuka-lwr/ics_lwr/ics_lwr_setup/enviroment/brick_pick_and_place_environment.urdf.xacro 	modified:   kuka-lwr/lwr_description/model/kuka_lwr.gazebo.xacro 	modified:   kuka-lwr/lwr_description/model/kuka_lwr.transmission.xacro 	modified:   kuka-lwr/lwr_description/model/kuka_lwr.urdf.xacro 	modified:   kuka-lwr/lwr_description/model/kuka_materials.xacro 	modified:   kuka-lwr/lwr_hw/include/lwr_hw/lwr_hw.h 	modified:   kuka-lwr/lwr_hw/include/lwr_hw/lwr_hw_gazebo.h 	modified:   kuka-lwr/lwr_hw/nodes/lwr_hw_gazebo_plugin.cpp 	modified:   kuka-lwr/lwr_hw/src/lwr_hw/lwr_hw.cpp

File: kuka-lwr/ics_lwr/ics_lwr_setup/enviroment/brick_pick_and_place_environment.urdf.xacro (robot description, xacro)
@@ -17,20 +17,20 @@
     <link name="world"/>
     <!-- table -->
-	<property name="world_origin_x" value="0.0" />
-	<property name="world_origin_y" value="0.0" />
-	<property name="world_origin_z" value="0.0" />
+	<xacro:property name="world_origin_x" value="0.0" />
+	<xacro:property name="world_origin_y" value="0.0" />
+	<xacro:property name="world_origin_z" value="0.0" />
 	<!-- table properties -->
-	<property name="table_height" value="0.878" />
-	<property name="table_width" value="1.0" />
-	<property name="table_depth" value="0.60" />
-	<property name="table_top_thickness" value="0.018"/>
-	<property name="table_origin_x" value="${world_origin_x + table_width/2}" />
-	<property name="table_origin_y" value="${world_origin_y + table_depth/2}" />
-	<property name="table_origin_z" value="${world_origin_z - table_top_thickness/2}" />
-	<property name="leg_edge" value="0.04" />
-	<property name="leg_pos_x" value="${leg_edge/2}" />
-	<property name="leg_pos_y" value="${leg_edge/2}" />
-	<property name="leg_height" value="${table_height - table_top_thickness}" />
-	<property name="leg_pos_z" value="${- table_top_thickness/2 - leg_height/2}" />
+	<xacro:property name="table_height" value="0.878" />
+	<xacro:property name="table_width" value="1.0" />
+	<xacro:property name="table_depth" value="0.60" />
+	<xacro:property name="table_top_thickness" value="0.018"/>
+	<xacro:property name="table_origin_x" value="${world_origin_x + table_width/2}" />
+	<xacro:property name="table_origin_y" value="${world_origin_y + table_depth/2}" />
+	<xacro:property name="table_origin_z" value="${world_origin_z - table_top_thickness/2}" />
+	<xacro:property name="leg_edge" value="0.04" />
+	<xacro:property name="leg_pos_x" value="${leg_edge/2}" />
+	<xacro:property name="leg_pos_y" value="${leg_edge/2}" />
+	<xacro:property name="leg_height" value="${table_height - table_top_thickness}" />
+	<xacro:property name="leg_pos_z" value="${- table_top_thickness/2 - leg_height/2}" />
 	<material name="table_color">
 		<!-- dark brown -->

File: kuka-lwr/lwr_description/model/kuka_lwr.gazebo.xacro (robot description, xacro)
@@ -1,4 +1,4 @@
 <?xml version="1.0"?>
-<robot xmlns:xacro="http://ros.org/wiki/xacro">
+<robot xmlns:xacro="http://www.ros.org/wiki/xacro">
 	<xacro:macro name="kuka_lwr_gazebo" params="name">
 		<gazebo>

File: kuka-lwr/lwr_description/model/kuka_lwr.transmission.xacro (robot description, xacro)
@@ -1,4 +1,4 @@
 <?xml version="1.0"?>
-<robot xmlns:xacro="http://ros.org/wiki/xacro">
+<robot xmlns:xacro="http://www.ros.org/wiki/xacro">
 	<xacro:property name="Interface10" value="PositionJointInterface"/>
 	<xacro:property name="Interface30" value="EffortJointInterface"/>

File: kuka-lwr/lwr_description/model/kuka_lwr.urdf.xacro (robot description, xacro)
@@ -15,9 +15,12 @@
         <xacro:property name="velocity_scale" value="0.15"/>
         <xacro:property name="effort_scale" value="1"/>
+        <xacro:property name="max_stiffness" value="5000"/>
+        <xacro:property name="min_stiffness" value="0"/>
+        <xacro:property name="rate_stiffness" value="20000"/> <!-- reflex to stiffness -->
 	<!-- URDF model /-->
 	<xacro:macro name="kuka_lwr" params="parent name *origin">
             <!-- First (shoulder) element of the arm. Fixed to its parent. -->
             <joint name="${parent}_${name}_base_joint" type="fixed">
-                <insert_block name="origin"/>
+                <xacro:insert_block name="origin"/>
                 <origin xyz="0 0 0" rpy="0 0 0"/>
                 <parent link="${parent}"/>

File: kuka-lwr/lwr_description/model/kuka_materials.xacro (robot description, xacro)
@@ -1,4 +1,4 @@
 <?xml version="1.0"?>
-<robot xmlns:xacro="http://ros.org/wiki/xacro">
+<robot xmlns:xacro="http://www.ros.org/wiki/xacro">
   <material name="Kuka/DarkGrey">
     <color rgba="0.3 0.3 0.3 1.0"/>
