Commit message: Added features coordinates filtering in visual_features_extractor iai_kinect2 added into meta package eye-to-hand Added aruco marker size parameter to kinect_fusion, changed  sensors TFs hri enviromental markers are modified, since the enviroment is new Modified joint limit for robot xacro Improvements in imbvs_with_obstacles_avoidance
	modified:   eye-in-hand/visual_features_extractor/CMakeLists.txt
	modified:   eye-in-hand/visual_features_extractor/include/visual_features_extractor/visual_features_extractor.h
	modified:   eye-in-hand/visual_features_extractor/launch/visual_features_extractor.launch
	modified:   eye-in-hand/visual_features_extractor/src/visual_features_extractor.cpp
	modified:   eye-to-hand/eye_to_hand/package.xml
	renamed:    iai_kinect2-master/LICENSE -> eye-to-hand/iai_kinect2-master/LICENSE
	renamed:    iai_kinect2-master/README.md -> eye-to-hand/iai_kinect2-master/README.md
	renamed:    iai_kinect2-master/iai_kinect2/CMakeLists.txt -> eye-to-hand/iai_kinect2-master/iai_kinect2/CMakeLists.txt
	renamed:    iai_kinect2-master/iai_kinect2/package.xml -> eye-to-hand/iai_kinect2-master/iai_kinect2/package.xml
	renamed:    iai_kinect2-master/kinect2_bridge/CMakeLists.txt -> eye-to-hand/iai_kinect2-master/kinect2_bridge/CMakeLists.txt
	renamed:    iai_kinect2-master/kinect2_bridge/README.md -> eye-to-hand/iai_kinect2-master/kinect2_bridge/README.md
	renamed:    iai_kinect2-master/kinect2_bridge/data/003722754847/calib_color.yaml -> eye-to-hand/iai_kinect2-master/kinect2_bridge/data/003722754847/calib_color.yaml
	renamed:    iai_kinect2-master/kinect2_bridge/data/003722754847/calib_color.yaml~ -> eye-to-hand/iai_kinect2-master/kinect2_bridge/data/003722754847/calib_color.yaml~
	renamed:    iai_kinect2-master/kinect2_bridge/data/003722754847/calib_depth.yaml -> eye-to-hand/iai_kinect2-master/kinect2_bridge/data/003722754847/calib_depth.yaml
	renamed:    iai_kinect2-master/kinect2_bridge/data/003722754847/calib_ir.yaml -> eye-to-hand/iai_kinect2-master/kinect2_bridge/data/003722754847/calib_ir.yaml
	renamed:    iai_kinect2-master/kinect2_bridge/data/003722754847/calib_pose.yaml -> eye-to-hand/iai_kinect2-master/kinect2_bridge/data/003722754847/calib_pose.yaml
	renamed:    iai_kinect2-master/kinect2_bridge/data/011296264147/calib_color.yaml -> eye-to-hand/iai_kinect2-master/kinect2_bridge/data/011296264147/calib_color.yaml
	renamed:    iai_kinect2-master/kinect2_bridge/data/011296264147/calib_depth.yaml -> eye-to-hand/iai_kinect2-master/kinect2_bridge/data/011296264147/calib_depth.yaml
	renamed:    iai_kinect2-master/kinect2_bridge/data/011296264147/calib_ir.yaml -> eye-to-hand/iai_kinect2-master/kinect2_bridge/data/011296264147/calib_ir.yaml
	renamed:    iai_kinect2-master/kinect2_bridge/data/011296264147/calib_pose.yaml -> eye-to-hand/iai_kinect2-master/kinect2_bridge/data/011296264147/calib_pose.yaml
	renamed:    iai_kinect2-master/kinect2_bridge/data/196605135147/calib_color.yaml -> eye-to-hand/iai_kinect2-master/kinect2_bridge/data/196605135147/calib_color.yaml
	renamed:    iai_kinect2-master/kinect2_bridge/data/196605135147/calib_depth.yaml -> eye-to-hand/iai_kinect2-master/kinect2_bridge/data/196605135147/calib_depth.yaml
	renamed:    iai_kinect2-master/kinect2_bridge/data/196605135147/calib_ir.yaml -> eye-to-hand/iai_kinect2-master/kinect2_bridge/data/196605135147/calib_ir.yaml
	renamed:    iai_kinect2-master/kinect2_bridge/data/196605135147/calib_pose.yaml -> eye-to-hand/iai_kinect2-master/kinect2_bridge/data/196605135147/calib_pose.yaml
	renamed:    iai_kinect2-master/kinect2_bridge/data/299150235147/calib_color.yaml -> eye-to-hand/iai_kinect2-master/kinect2_bridge/data/299150235147/calib_color.yaml
	renamed:    iai_kinect2-master/kinect2_bridge/data/299150235147/calib_ir.yaml -> eye-to-hand/iai_kinect2-master/kinect2_bridge/data/299150235147/calib_ir.yaml
	renamed:    iai_kinect2-master/kinect2_bridge/data/299150235147/calib_pose.yaml -> eye-to-hand/iai_kinect2-master/kinect2_bridge/data/299150235147/calib_pose.yaml
	renamed:    iai_kinect2-master/kinect2_bridge/data/old/003722754847/calib_color.yaml -> eye-to-hand/iai_kinect2-master/kinect2_bridge/data/old/003722754847/calib_color.yaml
	renamed:    iai_kinect2-master/kinect2_bridge/data/old/003722754847/calib_depth.yaml -> eye-to-hand/iai_kinect2-master/kinect2_bridge/data/old/003722754847/calib_depth.yaml
	renamed:    iai_kinect2-master/kinect2_bridge/data/old/003722754847/calib_ir.yaml -> eye-to-hand/iai_kinect2-master/kinect2_bridge/data/old/003722754847/calib_ir.yaml
	renamed:    iai_kinect2-master/kinect2_bridge/data/old/003722754847/calib_pose.yaml -> eye-to-hand/iai_kinect2-master/kinect2_bridge/data/old/003722754847/calib_pose.yaml
	renamed:    iai_kinect2-master/kinect2_bridge/data/old/011296264147/calib_color.yaml -> eye-to-hand/iai_kinect2-master/kinect2_bridge/data/old/011296264147/calib_color.yaml
	renamed:    iai_kinect2-master/kinect2_bridge/data/old/011296264147/calib_depth.yaml -> eye-to-hand/iai_kinect2-master/kinect2_bridge/data/old/011296264147/calib_depth.yaml
	renamed:    iai_kinect2-master/kinect2_bridge/data/old/011296264147/calib_ir.yaml -> eye-to-hand/iai_kinect2-master/kinect2_bridge/data/old/011296264147/calib_ir.yaml
	renamed:    iai_kinect2-master/kinect2_bridge/data/old/011296264147/calib_pose.yaml -> eye-to-hand/iai_kinect2-master/kinect2_bridge/data/old/011296264147/calib_pose.yaml
	renamed:    iai_kinect2-master/kinect2_bridge/include/kinect2_bridge/kinect2_definitions.h -> eye-to-hand/iai_kinect2-master/kinect2_bridge/include/kinect2_bridge/kinect2_definitions.h
	renamed:    iai_kinect2-master/kinect2_bridge/launch/kinect2_bridge.launch -> eye-to-hand/iai_kinect2-master/kinect2_bridge/launch/kinect2_bridge.launch
	renamed:    iai_kinect2-master/kinect2_bridge/launch/kinect2_bridge_k1.launch -> eye-to-hand/iai_kinect2-master/kinect2_bridge/launch/kinect2_bridge_k1.launch
	renamed:    iai_kinect2-master/kinect2_bridge/launch/kinect2_bridge_k2.launch -> eye-to-hand/iai_kinect2-master/kinect2_bridge/launch/kinect2_bridge_k2.launch
	renamed:    iai_kinect2-master/kinect2_bridge/nodelet_plugins.xml -> eye-to-hand/iai_kinect2-master/kinect2_bridge/nodelet_plugins.xml
	renamed:    iai_kinect2-master/kinect2_bridge/package.xml -> eye-to-hand/iai_kinect2-master/kinect2_bridge/package.xml
	renamed:    iai_kinect2-master/kinect2_bridge/src/kinect2_bridge.cpp -> eye-to-hand/iai_kinect2-master/kinect2_bridge/src/kinect2_bridge.cpp
	renamed:    iai_kinect2-master/kinect2_calibration/CMakeLists.txt -> eye-to-hand/iai_kinect2-master/kinect2_calibration/CMakeLists.txt
	renamed:    iai_kinect2-master/kinect2_calibration/README.md -> eye-to-hand/iai_kinect2-master/kinect2_calibration/README.md
	renamed:    iai_kinect2-master/kinect2_calibration/include/kinect2_calibration/kinect2_calibration_definitions.h -> eye-to-hand/iai_kinect2-master/kinect2_calibration/include/kinect2_calibration/kinect2_calibration_definitions.h
	renamed:    iai_kinect2-master/kinect2_calibration/package.xml -> eye-to-hand/iai_kinect2-master/kinect2_calibration/package.xml
	renamed:    iai_kinect2-master/kinect2_calibration/patterns/chess5x7x0.03.pdf -> eye-to-hand/iai_kinect2-master/kinect2_calibration/patterns/chess5x7x0.03.pdf
	renamed:    iai_kinect2-master/kinect2_calibration/patterns/chess5x7x0.03.svg -> eye-to-hand/iai_kinect2-master/kinect2_calibration/patterns/chess5x7x0.03.svg
	renamed:    iai_kinect2-master/kinect2_calibration/patterns/chess7x9x0.025.pdf -> eye-to-hand/iai_kinect2-master/kinect2_calibration/patterns/chess7x9x0.025.pdf
	renamed:    iai_kinect2-master/kinect2_calibration/patterns/chess7x9x0.025.svg -> eye-to-hand/iai_kinect2-master/kinect2_calibration/patterns/chess7x9x0.025.svg
	renamed:    iai_kinect2-master/kinect2_calibration/patterns/chess9x11x0.02.pdf -> eye-to-hand/iai_kinect2-master/kinect2_calibration/patterns/chess9x11x0.02.pdf
	renamed:    iai_kinect2-master/kinect2_calibration/patterns/chess9x11x0.02.svg -> eye-to-hand/iai_kinect2-master/kinect2_calibration/patterns/chess9x11x0.02.svg
	renamed:    iai_kinect2-master/kinect2_calibration/src/kinect2_calibration.cpp -> eye-to-hand/iai_kinect2-master/kinect2_calibration/src/kinect2_calibration.cpp
	renamed:    iai_kinect2-master/kinect2_registration/CMakeLists.txt -> eye-to-hand/iai_kinect2-master/kinect2_registration/CMakeLists.txt
	renamed:    iai_kinect2-master/kinect2_registration/README.md -> eye-to-hand/iai_kinect2-master/kinect2_registration/README.md
	renamed:    iai_kinect2-master/kinect2_registration/cmake/CheckOpenCLICDLoader.cmake -> eye-to-hand/iai_kinect2-master/kinect2_registration/cmake/CheckOpenCLICDLoader.cmake
	renamed:    iai_kinect2-master/kinect2_registration/cmake/FindOpenCL.cmake -> eye-to-hand/iai_kinect2-master/kinect2_registration/cmake/FindOpenCL.cmake
	renamed:    iai_kinect2-master/kinect2_registration/cmake/kinect2_registration.cmake.in -> eye-to-hand/iai_kinect2-master/kinect2_registration/cmake/kinect2_registration.cmake.in
	renamed:    iai_kinect2-master/kinect2_registration/include/internal/CL/cl.hpp -> eye-to-hand/iai_kinect2-master/kinect2_registration/include/internal/CL/cl.hpp
	renamed:    iai_kinect2-master/kinect2_registration/include/kinect2_registration/kinect2_console.h -> eye-to-hand/iai_kinect2-master/kinect2_registration/include/kinect2_registration/kinect2_console.h
	renamed:    iai_kinect2-master/kinect2_registration/include/kinect2_registration/kinect2_registration.h -> eye-to-hand/iai_kinect2-master/kinect2_registration/include/kinect2_registration/kinect2_registration.h
	renamed:    iai_kinect2-master/kinect2_registration/package.xml -> eye-to-hand/iai_kinect2-master/kinect2_registration/package.xml
	renamed:    iai_kinect2-master/kinect2_registration/src/depth_registration.cl -> eye-to-hand/iai_kinect2-master/kinect2_registration/src/depth_registration.cl
	renamed:    iai_kinect2-master/kinect2_registration/src/depth_registration_cpu.cpp -> eye-to-hand/iai_kinect2-master/kinect2_registration/src/depth_registration_cpu.cpp
	renamed:    iai_kinect2-master/kinect2_registration/src/depth_registration_cpu.h -> eye-to-hand/iai_kinect2-master/kinect2_registration/src/depth_registration_cpu.h
	renamed:    iai_kinect2-master/kinect2_registration/src/depth_registration_opencl.cpp -> eye-to-hand/iai_kinect2-master/kinect2_registration/src/depth_registration_opencl.cpp
	renamed:    iai_kinect2-master/kinect2_registration/src/depth_registration_opencl.h -> eye-to-hand/iai_kinect2-master/kinect2_registration/src/depth_registration_opencl.h
	renamed:    iai_kinect2-master/kinect2_registration/src/kinect2_registration.cpp -> eye-to-hand/iai_kinect2-master/kinect2_registration/src/kinect2_registration.cpp
	renamed:    iai_kinect2-master/kinect2_viewer/CMakeLists.txt -> eye-to-hand/iai_kinect2-master/kinect2_viewer/CMakeLists.txt
	renamed:    iai_kinect2-master/kinect2_viewer/README.md -> eye-to-hand/iai_kinect2-master/kinect2_viewer/README.md
	renamed:    iai_kinect2-master/kinect2_viewer/package.xml -> eye-to-hand/iai_kinect2-master/kinect2_viewer/package.xml
	renamed:    iai_kinect2-master/kinect2_viewer/src/viewer.cpp -> eye-to-hand/iai_kinect2-master/kinect2_viewer/src/viewer.cpp
	modified:   eye-to-hand/kinect_fusion/include/kinect_fusion/kinect_fusion.h
	modified:   eye-to-hand/kinect_fusion/launch/hri_kinect_fusion.launch
	modified:   eye-to-hand/kinect_fusion/launch/ics_kinect_fusion.launch
	modified:   eye-to-hand/kinect_fusion/nodes/kinect_fusion_node.cpp
	modified:   eye-to-hand/kinect_fusion/src/kinect_fusion.cpp
	modified:   eye-to-hand/obstacle_detector/config/hri_parameters.yaml
	modified:   eye-to-hand/obstacle_detector/nodes/obstacle_detector_node.cpp
	modified:   eye-to-hand/obstacle_detector/src/obstacle_detector.cpp
	modified:   imbvs_with_obstacles_avoidance/include/imbvs_with_obstacles_avoidance/imbvs_with_obstacles_avoidance.h
	modified:   imbvs_with_obstacles_avoidance/launch/imbvs_with_obstacles_avodance.launch
	modified:   imbvs_with_obstacles_avoidance/src/imbvs_with_obstacles_avoidance.cpp
	new file:   kuka-lwr/hri_lwr/hri_lwr_launch/launch/Clouds.rviz
	new file:   kuka-lwr/hri_lwr/hri_lwr_launch/launch/obstacles_only.rviz
	modified:   kuka-lwr/hri_lwr/hri_lwr_launch/launch/rviz_config.rviz
	new file:   kuka-lwr/ics_lwr/ics_lwr_launch/launch/Clouds.rviz
	modified:   kuka-lwr/lwr_description/model/kuka_lwr.urdf.xacro
	modified:   kuka-lwr/lwr_hw/src/fri/friremote.cpp

File: kuka-lwr/lwr_description/model/kuka_lwr.urdf.xacro (robot description, xacro)
@@ -79,9 +79,9 @@
                 </collision>
             </link>
-            <!-- Third segment of the arm. Joint along y-axis -->
+            <!-- Third segment of the arm. Joint along y-axis  <limit lower="${-120 * M_PI / 180}" upper="${120 * M_PI / 180}" for ics-->
             <joint name="${name}_a2_joint" type="revolute">
                     <origin xyz="0 0 0.2005" rpy="0 0 0"/>
                     <axis xyz="0 -1 0"/>
-                    <limit lower="${-120 * M_PI / 180}" upper="${120 * M_PI / 180}" effort="176" velocity="${velocity_scale * 110 * M_PI / 180}" />
+                    <limit lower="${-30 * M_PI / 180}" upper="${210 * M_PI / 180}" effort="176" velocity="${velocity_scale * 110 * M_PI / 180}" />
                     <dynamics friction="10.0" damping="1.0"/>
                     <parent link="${name}_a1_link"/>
@@ -223,5 +223,5 @@
                 <origin xyz="0 0 0.19" rpy="0 0 0"/>
                 <axis xyz="0 -1 0"/>
-                <limit lower="${-120 * M_PI / 180}" upper="${120 * M_PI / 180}" effort="38" velocity="${velocity_scale * 184 * M_PI / 180}" />
+                <limit lower="${-130 * M_PI / 180}" upper="${130 * M_PI / 180}" effort="38" velocity="${velocity_scale * 184 * M_PI / 180}" />
                 <dynamics friction="10.0" damping="1.0"/>
                 <parent link="${name}_a4_link"/>

Commit message: Changed joints limits. Fixed typo in imbvs_with_obstacles_avoidance

File: kuka-lwr/lwr_description/model/kuka_lwr.urdf.xacro (robot description, xacro)
@@ -83,5 +83,5 @@
                     <origin xyz="0 0 0.2005" rpy="0 0 0"/>
                     <axis xyz="0 -1 0"/>
-                    <limit lower="${-30 * M_PI / 180}" upper="${210 * M_PI / 180}" effort="176" velocity="${velocity_scale * 110 * M_PI / 180}" />
+                    <limit lower="${-170 * M_PI / 180}" upper="${170 * M_PI / 180}" effort="176" velocity="${velocity_scale * 110 * M_PI / 180}" />
                     <dynamics friction="10.0" damping="1.0"/>
                     <parent link="${name}_a1_link"/>
